Commit message: fixed friction can now turn scuffedly

File: install/ros_gz_example_description/share/ros_gz_example_description/models/diff_drive/rover_model.urdf (robot description, URDF)
Before this commit: robot diff_drive, 12 links, 11 joints
Links:
- link back_wheel_l: mass 0.8 -> 1.5
- link back_wheel_r: mass 0.8 -> 1.5
- link front_wheel_l: mass 0.8 -> 1.5; geometry collision cylinder length=0.067 radius=0.079; visual box size=0.04 0.04 0.001
- link front_wheel_r: mass 0.8 -> 1.5
Joints:
- joint bkwheel_to_leg_l: origin xyz=0.12 0 0.0565 rpy=0 0 1 -> xyz=0.12 0 0.0565 rpy=0 0 0

Commit message: fixed urdf wheel naming

File: install/ros_gz_example_description/share/ros_gz_example_description/models/diff_drive/rover_model.urdf (robot description, URDF)
Before this commit: robot diff_drive, 12 links, 11 joints
Links:
- link front_wheel_l: geometry collision cylinder length=0.067 radius=0.079; visual cylinder length=0.067 radius=0.079
- link front_wheel_r: geometry collision cylinder length=0.067 radius=0.079; visual box size=0.04 0.04 0.001
Joints:
- joint bkwheel_to_leg_l: child back_wheel_l -> back_wheel_r
- joint bkwheel_to_leg_r: child back_wheel_r -> back_wheel_l
- joint frwheel_to_leg_l: child front_wheel_l -> front_wheel_r
- joint frwheel_to_leg_r: child front_wheel_r -> front_wheel_l

Commit message: it can turn now yay just needs speed

File: install/ros_gz_example_description/share/ros_gz_example_description/models/diff_drive/rover_model.urdf (robot description, URDF)
Before this commit: robot diff_drive, 12 links, 11 joints
Links:
- link lidar_link: mass 0.1 -> 0.0
Joints:
- joint base_to_lleg: type revolute -> fixed
- joint base_to_rleg: type revolute -> fixed

Commit message: updated friction so turns are smoother

File: install/ros_gz_example_description/share/ros_gz_example_description/models/diff_drive/rover_model.urdf (robot description, URDF)
Before this commit: robot diff_drive, 12 links, 11 joints
Links:
- link back_wheel_l: mass 1.5 -> 1
- link back_wheel_r: mass 1.5 -> 1
- link front_wheel_l: mass 1.5 -> 1
- link front_wheel_r: mass 1.5 -> 1
